File: electronics/DeltaX_SAGA/DeltaX_SAGA.kicad_pcb (KiCad board)
At the start: 4 copper layers, 50 x 50 mm, 73 parts, among them J1 USB_B_Micro, J10 Motor3_Encoder, J11 M12, J12 M21, J13 M22, J14 M31, J15 M33, J16 Thrower+, J17 Thrower-, J2 Programmer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

Commit message: PCB design updated
Routing:
- net +5VD: track 15.8 -> 9.15 mm, vias 17 -> 8
- net GND2: track 79.9 -> 73.3 mm, vias 120 -> 111
- net GND: track 20.9 -> 15.0 mm, vias 42 -> 33
- net +3.3V: track 14.7 -> 10.1 mm, vias 30 -> 21

Commit message: PCB design updated
Parts:
- moved C4 14.3 mm to (163.0, 125.4), turned to -90 degrees
- moved C11 14.3 mm to (150.1, 119.2), turned to 180 degrees
- moved L1 7.33 mm to (133.4, 102.9), turned to 90 degrees
- moved C27 3.11 mm to (133.9, 95.1), turned to 0 degrees
- moved R1 2.52 mm to (143.6, 97.8), turned to -90 degrees
- moved R2 1.92 mm to (145.4, 97.3), turned to -90 degrees
- moved C23 1.47 mm to (147.3, 100.7)
- moved C26 1.47 mm to (143.2, 103.1)
- moved U5 1.47 mm to (143.7, 99.9)
- moved C24 1.47 mm to (145.3, 100.7)
- moved C25 1.31 mm to (141.9, 97.8), turned to 90 degrees
- moved C2 0.61 mm to (133.6, 111.0)
- moved C15 0.41 mm to (158.6, 111.1)
- moved C18 0.41 mm to (158.6, 106.1)
- moved C16 0.31 mm to (143.5, 111.0)
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Routing:
- net +3.3V: track 10.1 -> 18.8 mm, vias 21 -> 14
- net GND2: track 73.3 -> 65.2 mm, vias 111 -> 118
- net +5VD: track 9.15 -> 14.2 mm, vias 8 -> 5
- net /FB: track 8.54 -> 3.89 mm
- net GND: track 15.0 -> 17.6 mm
- net /Motor3_DIR_Isolated: track 21.6 -> 19.8 mm
- net /nSLEEP_Isolated: track 46.3 -> 44.8 mm, vias 5 -> 6
- net /Motor3_PWM_Isolated: track 22.0 -> 20.6 mm
- net /Motor1_PWM_Isolated: track 28.1 -> 28.7 mm
- net /Motor2_PWM_Isolated: track 27.6 -> 27.0 mm

Commit message: PCB design updated
Parts:
- L1: value 6.8uH -> 5.6uH
Changed lines of the file:
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@@
       (effects (font (size 0.3 0.3) (thickness 0.075)) (justify mirror))
     )
-    (fp_text value "6.8uH" (at 1.2464 7.0884 270 unlocked) (layer "B.Fab")
+    (fp_text value "5.6uH" (at 1.2464 7.0884 270 unlocked) (layer "B.Fab")
       (effects (font (size 0.5 0.5) (thickness 0.125)) (justify mirror))
     )

Commit message: PCB design updated
Parts:
- moved C11 14.8 mm to (159.6, 130.6), turned to 90 degrees
- moved R3 7.77 mm to (154.3, 99.9), turned to 90 degrees
- moved Q1 5.96 mm to (159.2, 99.2), turned to 90 degrees
- moved FB1 2.00 mm to (157.9, 130.6), turned to -90 degrees
- moved C1 1.32 mm to (150.8, 118.6), turned to -90 degrees
- moved R12 1.12 mm to (165.7, 92.9), turned to 90 degrees
- moved C30 0.08 mm to (164.4, 89.3)
- moved C33 0.08 mm to (166.6, 89.3)
- moved C14 0.08 mm to (162.2, 89.3)
- moved C21 0.08 mm to (160.0, 89.3)
- moved C36 0.08 mm to (157.8, 89.3)
Routing:
- net GND2: track 65.2 -> 23.1 mm, vias 118 -> 77
- net /Motor3_DIR_Isolated: track 19.8 -> 30.2 mm
- net /Motor3_PWM_Isolated: track 20.6 -> 30.7 mm
- net /VM: track 9.23 -> 0.83 mm, vias 17 -> 9
- net +3.3V: track 18.8 -> 16.3 mm, vias 14 -> 10
- net GND: track 17.6 -> 15.3 mm, vias 33 -> 26
- net /nSLEEP_Isolated: track 44.8 -> 46.5 mm
- net /Motor1_PWM_Isolated: track 28.7 -> 27.3 mm
- net /Motor1_DIR_Isolated: track 27.5 -> 26.4 mm
- net /USB_D-: track 12.1 -> 11.6 mm
- net /SWCLK: track 17.4 -> 16.9 mm
- net /USB_D+: track 12.2 -> 11.7 mm
- net /V+: vias 16 -> 12
Other:
- board text removed: "J7"

Commit message: PCB design updated
Connections:
- J3 pad 1: +5VD -> /Servo_PWM_Isolated
- J3 pad 2: /Servo_PWM_Isolated -> +5VD
Routing:
- net /Servo_PWM_Isolated: track 15.2 -> 21.8 mm
- net GND: track 15.3 -> 14.9 mm, vias 26 -> 25
Changed lines of the file:
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@@
     (fp_line (start 1.27 6.35) (end -1.27 6.35) (layer "F.Fab") (width 0.1))
     (pad "1" thru_hole rect (at 0 0) (size 2.5 1.75) (drill 0.8) (layers *.Cu *.Mask)
-      (net 78 "+5VD") (pinfunction "Pin_1") (pintype "passive"))
+      (net 54 "/Servo_PWM_Isolated") (pinfunction "Pin_1") (pintype "passive"))
     (pad "2" thru_hole oval (at 0 2.54) (size 2.5 1.75) (drill 0.8) (layers *.Cu *.Mask)
-      (net 54 "/Servo_PWM_Isolated") (pinfunction "Pin_2") (pintype "passive"))
+      (net 78 "+5VD") (pinfunction "Pin_2") (pintype "passive"))
     (pad "3" thru_hole oval (at 0 5.08) (size 2.5 1.75) (drill 0.8) (layers *.Cu *.Mask)
       (net 5 "GND2") (pinfunction "Pin_3") (pintype "passive"))
@@
   (segment (start 147.32 94.4118) (end 148.8694 95.9612) (width 0.254) (layer "F.Cu") (net 52))
   (segment (start 136.652 94.4118) (end 147.32 94.4118) (width 0.25) (layer "F.Cu") (net 52))
+  (segment (start 131.1656 101.4984) (end 127.9484 101.4984) (width 0.25) (layer "F.Cu") (net 54))
+  (segment (start 127.9484 101.4984) (end 126.94 100.49) (width 0.25) (layer "F.Cu") (net 54))
+  (segment (start 136.525 102.8192) (end 132.4864 102.8192) (width 0.25) (layer "F.Cu") (net 54))
+  (segment (start 132.4864 102.8192) (end 131.1656 101.4984) (width 0.25) (layer "F.Cu") (net 54))
+  (segment (start 126.94 95.3) (end 127.5234 94.7166) (width 0.25) (layer "F.Cu") (net 54))
   (segment (start 137.3378 103.6441) (end 137.3378 103.632) (width 0.25) (layer "F.Cu") (net 54))
-  (segment (start 131.8768 102.2096) (end 132.4864 102.8192) (width 0.25) (layer "F.Cu") (net 54))
-  (segment (start 136.525 102.8192) (end 135.3566 102.8192) (width 0.25) (layer "F.Cu") (net 54))
-  (segment (start 131.1656 99.7204) (end 131.1656 101.4984) (width 0.25) (layer "F.Cu") (net 54))
-  (segment (start 133.6294 102.8192) (end 135.3566 102.8192) (width 0.25) (layer "F.Cu") (net 54))
-  (segment (start 130.2258 97.2566) (end 130.937 97.9678) (width 0.25) (layer "F.Cu") (net 54))
-  (segment (start 132.4864 102.8192) (end 133.6294 102.8192) (width 0.25) (layer "F.Cu") (net 54))
-  (segment (start 131.1656 101.4984) (end 131.8768 102.2096) (width 0.25) (layer "F.Cu") (net 54))
-  (segment (start 129.1336 97.2566) (end 130.2258 97.2566) (width 0.25) (layer "F.Cu") (net 54))
-  (segment (start 137.3378 103.632) (end 136.525 102.8192) (width 0.25) (layer "F.Cu") (net 54))
-  (segment (start 131.1656 98.1964) (end 131.1656 99.7204) (width 0.25) (layer "F.Cu") (net 54))
+  (segment (start 127.5234 94.7166) (end 129.1336 94.7166) (width 0.25) (layer "F.Cu") (net 54))
   (segment (start 137.3378 106.0868) (end 137.3378 105.3338) (width 0.25) (layer "F.Cu") (net 54))
-  (segment (start 130.937 97.9678) (end 131.1656 98.1964) (width 0.25) (layer "F.Cu") (net 54))
+  (segment (start 126.94 100.49) (end 126.94 95.3) (width 0.25) (layer "F.Cu") (net 54))
+  (segment (start 137.3378 103.632) (end 136.525 102.8192) (width 0.25) (layer "F.Cu") (net 54))
   (via (at 137.3378 103.6441) (size 0.45) (drill 0.2) (layers "F.Cu" "B.Cu") (net 54))
   (via (at 137.3378 105.3338) (size 0.45) (drill 0.2) (layers "F.Cu" "B.Cu") (net 54))
@@
   (segment (start 167.1574 129.6924) (end 167.2844 129.5654) (width 0.25) (layer "F.Cu") (net 68))
   (segment (start 140.7384 118.0592) (end 139.6492 118.0592) (width 0.25) (layer "F.Cu") (net 68))
-  (segment (start 167.4368 118.6368) (end 167.4368 119.0752) (width 0.2) (layer "F.Cu") (net 68))
   (segment (start 140.7384 116.7892) (end 139.6238 116.7892) (width 0.25) (layer "F.Cu") (net 68))
   (segment (start 162.8902 121.793) (end 162.828503 121.854697) (width 0.25) (layer "F.Cu") (net 68))
@@
   (via (at 154.1272 115.9764) (size 0.45) (drill 0.2) (layers "F.Cu" "B.Cu") (net 68))
   (via (at 150.5712 119.634) (size 0.45) (drill 0.2) (layers "F.Cu" "B.Cu") (net 68))
-  (via (at 167.4368 119.0752) (size 0.45) (drill 0.2) (layers "F.Cu" "B.Cu") (net 68))
   (via (at 160.147 127.801903) (size 0.45) (drill 0.2) (layers "F.Cu" "B.Cu") (net 68))
   (via (at 157.3276 127.878103) (size 0.45) (drill 0.2) (layers "F.Cu" "B.Cu") (net 68))

Commit message: PCB design added
Parts:
- moved R4 1.44 mm to (165.7, 129.0), turned to 90 degrees
- moved C7 1.12 mm to (169.5, 124.0)
- moved U2 1.12 mm to (166.8, 124.1)
- moved D1 0.97 mm to (164.1, 129.0), turned to 90 degrees
- moved C10 0.73 mm to (167.7, 128.7)
- moved J4 0.38 mm to (135.2, 85.1)
Routing:
- net +5V: track 0.86 -> 0.00 mm
- net +3.3V: vias 10 -> 11

Commit message: PCB design updated
Parts:
- J10: value Motor3_Encoder -> M3_Encoder
- J6: value Thrower Signal -> Thrower
- J8: value Motor1_Encoder -> M1_Encoder
- J9: value Motor2_Encoder -> M2_Encoder
- moved J6 0.27 mm to (129.1, 104.3)
Changed lines of the file:
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@@
       (effects (font (size 1 1) (thickness 0.2)))
     )
-    (fp_text value "Motor1_Encoder" (at -1.9403 -2.8415 90) (layer "F.SilkS")
-      (effects (font (size 0.7 0.7) (thickness 0.12)))
+    (fp_text value "M1_Encoder" (at -3.1727 -2.9751 90) (layer "F.SilkS")
+      (effects (font (size 1 1) (thickness 0.2)))
     )
     (fp_line (start 1.645 2.9) (end 1.645 3.87) (layer "F.SilkS") (width 0.127))
@@
   )
   (footprint "Micro-MaTch215079-4:TE_7-215079-4" (layer "F.Cu")
-    (at 128.8509 104.2571 90)
+    (at 129.1215 104.2675 90)
     (property "Sheetfile" "DeltaX_SAGA.kicad_sch")
     (property "Sheetname" "")
     (attr through_hole)
-    (fp_text reference "J6" (at -6.5929 -0.7609 180) (layer "F.SilkS")
+    (fp_text reference "J6" (at -6.5425 0.4185 180) (layer "F.SilkS")
       (effects (font (size 1 1) (thickness 0.2)))
     )
-    (fp_text value "Thrower Signal" (at -4.5565 -2.1303 90) (layer "F.SilkS")
-      (effects (font (size 0.7 0.7) (thickness 0.15)))
+    (fp_text value "Thrower" (at -3.4325 -2.3915 90) (layer "F.SilkS")
+      (effects (font (size 1 1) (thickness 0.2)))
     )
     (fp_line (start 1.645 -1.33) (end 1.645 0.7) (layer "F.SilkS") (width 0.127))
@@
       (effects (font (size 1 1) (thickness 0.2)))
     )
-    (fp_text value "SERVO" (at -2.4384 3.0226 90) (layer "F.SilkS")
-      (effects (font (size 0.6 0.6) (thickness 0.15)))
+    (fp_text value "SERVO" (at -2.2936 3.0134 90) (layer "F.SilkS")
+      (effects (font (size 1 1) (thickness 0.2)))
     )
     (fp_text user "${REFERENCE}" (at 0 2.54 90) (layer "F.Fab")
@@
       (effects (font (size 1 1) (thickness 0.2)))
     )
-    (fp_text value "Motor3_Encoder" (at -1.7117 -2.7145) (layer "F.SilkS")
-      (effects (font (size 0.7 0.7) (thickness 0.12)))
+    (fp_text value "M3_Encoder" (at -1.8417 -3.1427) (layer "F.SilkS")
+      (effects (font (size 1 1) (thickness 0.2)))
     )
     (fp_line (start 1.645 2.9) (end 1.645 3.87) (layer "F.SilkS") (width 0.127))
@@
       (effects (font (size 1 1) (thickness 0.2)))
     )
-    (fp_text value "Motor2_Encoder" (at -1.7018 -2.8448) (layer "F.SilkS")
-      (effects (font (size 0.7 0.7) (thickness 0.12)))
+    (fp_text value "M2_Encoder" (at -1.598 -3.0014) (layer "F.SilkS")
+      (effects (font (size 1 1) (thickness 0.2)))
     )
     (fp_line (start 1.645 2.9) (end 1.645 3.87) (layer "F.SilkS") (width 0.127))
@@
   (segment (start 151.9428 113.6396) (end 151.0284 112.7252) (width 0.25) (layer "F.Cu") (net 37))
   (segment (start 154.2288 113.6396) (end 151.9428 113.6396) (width 0.25) (layer "F.Cu") (net 37))
+  (segment (start 136.0678 103.4796) (end 134.0996 103.4796) (width 0.25) (layer "F.Cu") (net 41))
   (segment (start 148.4884 106.11) (end 148.4884 105.1052) (width 0.25) (layer "F.Cu") (net 41))
-  (segment (start 136.0678 103.4796) (end 133.4384 103.4796) (width 0.25) (layer "F.Cu") (net 41))
+  (segment (start 134.0996 103.4796) (end 133.7194 103.4796) (width 0.25) (layer "F.Cu") (net 41))
   (segment (start 136.9568 104.3686) (end 136.0678 103.4796) (width 0.25) (layer "F.Cu") (net 41))
   (segment (start 147.7518 104.3686) (end 136.9568 104.3686) (width 0.25) (layer "F.Cu") (net 41))
+  (segment (start 133.7194 103.4796) (end 131.6615 105.5375) (width 0.25) (layer "F.Cu") (net 41))
   (segment (start 148.4884 105.1052) (end 147.7518 104.3686) (width 0.25) (layer "F.Cu") (net 41))
-  (segment (start 133.4384 103.4796) (end 131.3909 105.5271) (width 0.25) (layer "F.Cu") (net 41))
   (segment (start 149.7584 104.2162) (end 150.0378 103.9368) (width 0.25) (layer "F.Cu") (net 42))
   (segment (start 157.872999 91.248799) (end 158.7754 92.1512) (width 0.25) (layer "F.Cu") (net 42))
@@
   (segment (start 147.32 94.4118) (end 148.8694 95.9612) (width 0.254) (layer "F.Cu") (net 52))
   (segment (start 136.652 94.4118) (end 147.32 94.4118) (width 0.25) (layer "F.Cu") (net 52))
-  (segment (start 131.1656 101.4984) (end 127.9484 101.4984) (width 0.25) (layer "F.Cu") (net 54))
-  (segment (start 127.9484 101.4984) (end 126.94 100.49) (width 0.25) (layer "F.Cu") (net 54))
-  (segment (start 136.525 102.8192) (end 132.4864 102.8192) (width 0.25) (layer "F.Cu") (net 54))
-  (segment (start 132.4864 102.8192) (end 131.1656 101.4984) (width 0.25) (layer "F.Cu") (net 54))
-  (segment (start 126.94 95.3) (end 127.5234 94.7166) (width 0.25) (layer "F.Cu") (net 54))
-  (segment (start 137.3378 103.6441) (end 137.3378 103.632) (width 0.25) (layer "F.Cu") (net 54))
-  (segment (start 127.5234 94.7166) (end 129.1336 94.7166) (width 0.25) (layer "F.Cu") (net 54))
+  (segment (start 129.1336 94.7166) (end 127.5234 94.7166) (width 0.25) (layer "F.Cu") (net 54))
+  (segment (start 136.525 102.8192) (end 137.3378 103.632) (width 0.25) (layer "F.Cu") (net 54))
+  (segment (start 127.9484 101.4984) (end 131.6584 101.4984) (width 0.25) (layer "F.Cu") (net 54))
+  (segment (start 126.94 95.3) (end 126.94 100.49) (width 0.25) (layer "F.Cu") (net 54))
+  (segment (start 137.3378 103.632) (end 137.3378 103.6441) (width 0.25) (layer "F.Cu") (net 54))
+  (segment (start 126.94 100.49) (end 127.9484 101.4984) (width 0.25) (layer "F.Cu") (net 54))
+  (segment (start 131.6584 101.4984) (end 132.9792 102.8192) (width 0.25) (layer "F.Cu") (net 54))
+  (segment (start 127.5234 94.7166) (end 126.94 95.3) (width 0.25) (layer "F.Cu") (net 54))
   (segment (start 137.3378 106.0868) (end 137.3378 105.3338) (width 0.25) (layer "F.Cu") (net 54))
-  (segment (start 126.94 100.49) (end 126.94 95.3) (width 0.25) (layer "F.Cu") (net 54))
-  (segment (start 137.3378 103.632) (end 136.525 102.8192) (width 0.25) (layer "F.Cu") (net 54))
+  (segment (start 132.9792 102.8192) (end 136.525 102.8192) (width 0.25) (layer "F.Cu") (net 54))
   (via (at 137.3378 103.6441) (size 0.45) (drill 0.2) (layers "F.Cu" "B.Cu") (net 54))
   (via (at 137.3378 105.3338) (size 0.45) (drill 0.2) (layers "F.Cu" "B.Cu") (net 54))

Commit message: PCB design updated
Parts:
- moved R2 0.48 mm to (145.0, 97.6)
- moved C25 0.31 mm to (141.6, 97.9)
- moved R1 0.30 mm to (143.3, 97.8)
